File: hardware/entrance-remote-pcb/layouts/default/default.kicad_pcb (KiCad board)
At the start: 2 copper layers, 40 parts

Commit message: feat(hardware): physical layout, procedural routing, 0 DRC violations and 3D CAD models for entrance-remote-pcb
Parts:
- D1, D2, D3, D4, D5, D6, D7: footprint entrance-remote-pcb:D_DO-201AD_P15.24mm_Horizontal -> entrance-remote-pcb:D_SOD-123
- moved R10 385.6 mm to (4.50, 8.00), turned to 90 degrees
- moved D8 380.1 mm to (0.00, 8.00), turned to -90 degrees
- moved C7 366.4 mm to (-5.00, -32.0)
- moved C8 366.4 mm to (5.00, -32.0), turned to 180 degrees
- moved J1 351.5 mm to (0.00, -32.0)
- moved D7 334.7 mm to (6.00, 22.0), turned to 180 degrees
- moved C10 328.5 mm to (-17.0, 31.0), turned to 180 degrees
- moved C11 324.2 mm to (6.00, 12.0), turned to 180 degrees
- moved R8 318.9 mm to (-17.0, 35.0)
- moved R9 314.5 mm to (6.00, 17.0)
- moved C9 304.1 mm to (-12.5, 31.0), turned to 180 degrees
- moved R7 294.6 mm to (-12.5, 35.0)
- moved SW7 279.1 mm to (-7.50, 29.5)
- moved D2 255.7 mm to (-35.0, -19.0), turned to 180 degrees
- moved C2 241.4 mm to (-30.5, -21.0)
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Connections:
- C1 pad 1: 2-1 -> 1
- C11 pad 1: 2-2 -> 1-6
- C2 pad 1: 1 -> 1-1
- C3 pad 1: mcu_sense -> 1-2
- C4 pad 1: mcu_sense-1 -> 1-3
- C5 pad 1: mcu_sense-2 -> 1-4
- C6 pad 1: mcu_sense-3 -> 1-5
- D1 pad 1: wakeup_bus -> 1
- D1 pad 2: 2-1 -> wakeup_bus
- D2 pad 1: wakeup_bus -> 1-1
- D2 pad 2: 1 -> wakeup_bus
- D3 pad 1: wakeup_bus -> 1-2
- D3 pad 2: mcu_sense -> wakeup_bus
- D4 pad 1: wakeup_bus -> 1-3
- D4 pad 2: mcu_sense-1 -> wakeup_bus
- D5 pad 1: wakeup_bus -> 1-4
- D5 pad 2: mcu_sense-2 -> wakeup_bus
- D6 pad 1: wakeup_bus -> 1-5
- D6 pad 2: mcu_sense-3 -> wakeup_bus
- D7 pad 1: wakeup_bus -> 1-6
- D7 pad 2: 2-2 -> wakeup_bus
- J2 pad 4: mcu_sense -> 1-2
- J2 pad 5: mcu_sense-1 -> 1-3
- J2 pad 6: mcu_sense-2 -> 1-4
- J2 pad 7: mcu_sense-3 -> 1-5
- J3 pad 1: 1 -> 1-1
- J3 pad 2: 2-1 -> 1
- J3 pad 3: 2-2 -> 1-6
- R1 pad 2: 2-1 -> 1
- R2 pad 2: 1 -> 1-1
- R3 pad 2: mcu_sense -> 1-2
- R4 pad 2: mcu_sense-1 -> 1-3
- R5 pad 2: mcu_sense-2 -> 1-4
- R6 pad 2: mcu_sense-3 -> 1-5
- R9 pad 2: 2-2 -> 1-6
- SW1 pad 1: 2-1 -> 1
- SW2 pad 1: 1 -> 1-1
- SW3 pad 1: mcu_sense -> 1-2
- SW4 pad 1: mcu_sense-1 -> 1-3
- SW5 pad 1: mcu_sense-2 -> 1-4
- SW6 pad 1: mcu_sense-3 -> 1-5
- SW7 pad S1: 2-2 -> 1-6
Routing:
- net vcc: track 0.00 -> 284.4 mm, vias 0 -> 12
- net wakeup_bus: track 0.00 -> 257.0 mm, vias 0 -> 8
- net 1-3: track 0.00 -> 84.8 mm, vias 0 -> 2
- net 1-1: track 0.00 -> 82.8 mm, vias 0 -> 3
- net 1-5: track 0.00 -> 81.9 mm, vias 0 -> 1
- net 1-2: track 0.00 -> 67.0 mm
- net B: track 0.00 -> 66.0 mm
- net 1-4: track 0.00 -> 53.1 mm
- net 1-6: track 0.00 -> 52.3 mm
- net A: track 0.00 -> 48.9 mm
- net 1: track 0.00 -> 48.1 mm
- net anode: track 0.00 -> 26.7 mm
- net 2: track 0.00 -> 6.64 mm, vias 0 -> 11
- net cathode: track 0.00 -> 4.53 mm
- added copper zone on B.Cu, net 2
- added copper zone on F.Cu, net 2
Other:
- board outline added: 80 x 80 mm
