File: hardware/cockpit-pcb/layouts/default/default.kicad_pcb (KiCad board)
At the start: 2 copper layers, 29 parts

Commit message: feat(hardware): physical layout, procedural routing, 0 DRC violations and 3D CAD models for cockpit-pcb
Parts:
- D1, D2, D3, D4, D5, D6: footprint cockpit-pcb:D_DO-201AD_P15.24mm_Horizontal -> cockpit-pcb:D_SOD-123
- moved C2 281.6 mm to (-21.5, -8.00)
- moved C1 271.7 mm to (-21.5, -11.0)
- moved R7 263.5 mm to (16.5, -4.38)
- moved J1 258.1 mm to (-17.5, -17.0)
- moved D7 257.0 mm to (13.0, -4.38)
- moved J4 220.9 mm to (-10.2, 17.5), turned to 180 degrees
- moved J5 216.9 mm to (3.81, 17.5), turned to 180 degrees
- moved J6 212.9 mm to (17.8, 17.5), turned to 180 degrees
- moved D6 187.5 mm to (12.7, 9.00), turned to 180 degrees
- moved C8 177.7 mm to (12.7, 12.0), turned to 180 degrees
- moved R6 167.4 mm to (12.7, 6.00)
- moved D5 152.5 mm to (17.8, 9.00), turned to 180 degrees
- moved C7 142.7 mm to (17.8, 12.0), turned to 180 degrees
- moved D4 141.6 mm to (-1.27, 9.00), turned to 180 degrees
- moved R5 132.3 mm to (17.8, 6.00)
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Connections:
- C3 pad 1: 2 -> 1
- C5 pad 1: mcu_sense-1 -> 1-1
- C6 pad 1: mcu_sense-2 -> mcu_sense-1
- C7 pad 1: mcu_sense-3 -> 1-2
- C8 pad 1: mcu_sense-4 -> mcu_sense-2
- D1 pad 1: wakeup_bus -> 1
- D1 pad 2: 2 -> wakeup_bus
- D2 pad 1: wakeup_bus -> mcu_sense
- D2 pad 2: mcu_sense -> wakeup_bus
- D3 pad 1: wakeup_bus -> 1-1
- D3 pad 2: mcu_sense-1 -> wakeup_bus
- D4 pad 1: wakeup_bus -> mcu_sense-1
- D4 pad 2: mcu_sense-2 -> wakeup_bus
- D5 pad 1: wakeup_bus -> 1-2
- D5 pad 2: mcu_sense-3 -> wakeup_bus
- D6 pad 1: wakeup_bus -> mcu_sense-2
- D6 pad 2: mcu_sense-4 -> wakeup_bus
- J2 pad 2: 2 -> 1
- J2 pad 4: mcu_sense-1 -> 1-1
- J2 pad 5: mcu_sense-2 -> mcu_sense-1
- J2 pad 6: mcu_sense-3 -> 1-2
- J2 pad 7: mcu_sense-4 -> mcu_sense-2
- J4 pad 1: 2 -> 1
- J5 pad 1: mcu_sense-1 -> 1-1
- J5 pad 3: mcu_sense-2 -> mcu_sense-1
- J6 pad 1: mcu_sense-3 -> 1-2
- J6 pad 3: mcu_sense-4 -> mcu_sense-2
- R1 pad 2: 2 -> 1
- R3 pad 2: mcu_sense-1 -> 1-1
- R4 pad 2: mcu_sense-2 -> mcu_sense-1
- R5 pad 2: mcu_sense-3 -> 1-2
- R6 pad 2: mcu_sense-4 -> mcu_sense-2
Routing:
- net vcc: track 0.00 -> 100.8 mm, vias 0 -> 7
- net gnd: track 0.00 -> 84.0 mm, vias 0 -> 17
- net wakeup_bus: track 0.00 -> 66.0 mm, vias 0 -> 9
- net 1-2: track 0.00 -> 57.8 mm, vias 0 -> 2
- net mcu_sense-2: track 0.00 -> 47.2 mm, vias 0 -> 2
- net 1-1: track 0.00 -> 35.8 mm, vias 0 -> 1
- net mcu_sense: track 0.00 -> 32.8 mm, vias 0 -> 1
- net 1: track 0.00 -> 30.2 mm
- net mcu_sense-1: track 0.00 -> 28.2 mm, vias 0 -> 1
- net anode: track 0.00 -> 4.44 mm
- net cathode: track 0.00 -> 1.65 mm
- added copper zone on B.Cu, net gnd
- added copper zone on F.Cu, net gnd
Other:
- board outline added: 55 x 45 mm
