File: hardware/central-pcb/layouts/default/default.kicad_pcb (KiCad board)
At the start: 2 copper layers, 58 parts

Commit message: feat(hardware): physical layout, procedural routing, 0 DRC violations and 3D CAD models for central-pcb
Parts:
- removed J17, J18, J19, J20: , central-pcb:PinSocket_1x02_P2.54mm_Vertical
- removed J2, J22, J3: , central-pcb:TerminalBlock_Phoenix_MPT-0,5-2-2.54_1x02_P2.54mm_Horizontal
- removed J21: , central-pcb:TerminalBlock_Phoenix_MPT-0,5-4-2.54_1x04_P2.54mm_Horizontal
- removed Q3, Q4, Q6: , central-pcb:SOT-23
- removed Q5: , central-pcb:SOIC-8_3.9x4.9mm_P1.27mm
- removed R4, R5, R6, R7, R8, R9: , central-pcb:R_0805_2012Metric
- removed U2, U3: , central-pcb:SOT-223
- added R19: , central-pcb:R_0805_2012Metric, F.Cu at (-42.0, 4.00)
- added R20: , central-pcb:R_0805_2012Metric, F.Cu at (-38.0, 4.00)
- added R21: , central-pcb:R_0805_2012Metric, F.Cu at (-44.5, 4.00)
- added R22: , central-pcb:R_0805_2012Metric, F.Cu at (-26.0, 4.00)
- added R23: , central-pcb:R_0805_2012Metric, F.Cu at (-22.0, 4.00)
- added R24: , central-pcb:R_0805_2012Metric, F.Cu at (-28.5, 4.00)
- added R25: , central-pcb:R_0805_2012Metric, F.Cu at (26.0, 4.00)
- added R26: , central-pcb:R_0805_2012Metric, F.Cu at (30.0, 4.00)
- added R27: , central-pcb:R_0805_2012Metric, F.Cu at (23.5, 4.00)
- added R28: , central-pcb:R_0805_2012Metric, F.Cu at (-17.0, -22.0)
- added R29: , central-pcb:R_0805_2012Metric, F.Cu at (42.0, 4.00)
- added R30: , central-pcb:R_0805_2012Metric, F.Cu at (46.0, 4.00)
- added R31: , central-pcb:R_0805_2012Metric, F.Cu at (39.5, 4.00)
- added R32: , central-pcb:R_0805_2012Metric, F.Cu at (-17.0, -1.68)
- added R33: , central-pcb:R_0805_2012Metric, F.Cu at (22.0, -18.0)
- added R34: , central-pcb:R_0805_2012Metric, F.Cu at (26.0, -18.0)
- added R35: , central-pcb:R_0805_2012Metric, F.Cu at (17.0, -14.4)
- added U10: , central-pcb:SOIC-14-1EP_3.9x8.7mm_P1.27mm_EP4.3x4.7mm, F.Cu at (42.0, 14.0)
- added U7: , central-pcb:SOIC-14-1EP_3.9x8.7mm_P1.27mm_EP4.3x4.7mm, F.Cu at (-42.0, 14.0)
- added U8: , central-pcb:SOIC-14-1EP_3.9x8.7mm_P1.27mm_EP4.3x4.7mm, F.Cu at (-26.0, 14.0)
- added U9: , central-pcb:SOIC-14-1EP_3.9x8.7mm_P1.27mm_EP4.3x4.7mm, F.Cu at (26.0, 14.0)
- J15: footprint central-pcb:PinSocket_1x05_P2.54mm_Vertical -> central-pcb:TerminalBlock_Phoenix_MPT-0,5-4-2.54_1x04_P2.54mm_Horizontal
- J16: footprint central-pcb:PinSocket_1x02_P2.54mm_Vertical -> central-pcb:TerminalBlock_Phoenix_MPT-0,5-2-2.54_1x02_P2.54mm_Horizontal
- Q2: footprint central-pcb:SOT-23 -> central-pcb:SOIC-8_3.9x4.9mm_P1.27mm
- U1, U6: footprint central-pcb:SOT-223 -> central-pcb:SOIC-14-1EP_3.9x8.7mm_P1.27mm_EP4.3x4.7mm
- moved R16 360.9 mm to (-58.0, 4.00), turned to -90 degrees
- moved J11 343.3 mm to (-58.0, 35.0)
- moved J13 313.9 mm to (-26.0, 35.0)
- moved J12 311.9 mm to (-42.0, 35.0)
- moved J6 302.1 mm to (34.0, -36.0), turned to 180 degrees
- moved R13 298.4 mm to (35.0, -16.0)
- moved D3 294.7 mm to (-22.0, -22.0), turned to 180 degrees
- moved D5 293.6 mm to (-22.0, -1.68), turned to 180 degrees
- moved J9 261.0 mm to (62.0, -14.0)
- moved U4 253.5 mm to (26.4, -25.0)
- moved J14 249.0 mm to (26.0, 35.0)
- moved D1 246.6 mm to (22.0, -11.8)
- moved J10 238.4 mm to (54.0, -36.0), turned to 180 degrees
- moved D4 236.5 mm to (47.1, 28.0), turned to 180 degrees
- moved U6 231.7 mm to (-58.0, 14.0), turned to -90 degrees
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Connections:
- C1 pad 1: v_out -> voltage_sensor-1
- C1 pad 2: 2 -> gnd
- D1 pad 2: 2 -> gnd
- D2 pad 2: 2 -> gnd
- D3 pad 2: 2 -> gnd
- D4 pad 1: 1-4 -> cathode
- D4 pad 2: 2 -> gnd
- D5 pad 2: 2 -> gnd
- J1 pad 2: 2 -> gnd
- J11 pad 1: out1_neg -> power_out-3
- J11 pad 2: 2 -> power_in
- J11 pad 4: power_in -> gnd
- J12 pad 1: out2_neg -> power_out-4
- J12 pad 2: 2 -> power_in
- J12 pad 4: power_in -> gnd
- J13 pad 1: out3_neg -> power_out-5
- J13 pad 2: 2 -> power_in
- J13 pad 4: power_in -> gnd
- J14 pad 1: out4_neg -> power_out-6
- J14 pad 2: 2 -> power_in
- J14 pad 4: power_in -> gnd
- J15 pad 1: 2 -> power_out-7
- J15 pad 2: GPIO12 -> power_in
- J15 pad 3: GPIO13 -> cathode
- J15 pad 4: GPIO14 -> gnd
- J16 pad 1: out1_pos -> power_in
- J16 pad 2: out1_neg -> gnd
- J4 pad 2: 2 -> gnd
- J5 pad 2: 2 -> gnd
- J7 pad 10: GPIO17 -> control-8
- J7 pad 11: GPIO18 -> control-3
- J7 pad 18: GPIO12 -> control-4
- J7 pad 19: GPIO13 -> control-5
- J7 pad 2: esp32.left_header-2 -> 2
- J7 pad 20: GPIO14 -> control-6
- J7 pad 21: 21 -> v_mcu_5v
- J7 pad 22: 2 -> gnd
- J7 pad 4: control-6 -> control-10
- J7 pad 8: GPIO15 -> control-7
- J8 pad 1: v_mcu_5v -> gnd
- J8 pad 18: 18 -> control-9
- J8 pad 19: control-5 -> 19
- J8 pad 2: 2 -> esp32.right_header-2
- J8 pad 20: control-3 -> 20
- J8 pad 21: control-4 -> gnd
- J8 pad 22: 2 -> gnd
- J8 pad 4: 4 -> v_out
- J8 pad 5: v_out -> 1
- J8 pad 6: 1 -> 6
- J9 pad 2: 2 -> gnd
- Q1 pad 2: 2 -> gnd
- Q2 pad 1: aux2_stage-gate -> power_in
- Q2 pad 2: 2 -> power_in
- Q2 pad 3: aux2_stage-drain -> power_in
- R1 pad 2: gate -> input
- R10 pad 1: control-4 -> 1
- R10 pad 2: 2 -> anode
- R11 pad 1: fan_stage-drain -> control-3
- R11 pad 2: power_in -> dcdc_opto-anode
- R12 pad 1: control-5 -> control-8
- R12 pad 2: inverter_opto-anode -> gate
- R13 pad 1: 1-2 -> control-8
- R13 pad 2: anode-1 -> gnd
- R14 pad 1: control-6 -> drain
- R14 pad 2: pump_stage-gate -> power_in
- R15 pad 1: control-6 -> control-9
- R15 pad 2: 2 -> inverter_opto-anode
- R16 pad 1: 1-1 -> control-4
- R16 pad 2: anode-2 -> led_zone1_stage-input
- R17 pad 1: power_in -> control-4
- R17 pad 2: v_out -> gnd
- R18 pad 1: v_out -> led_zone1_stage-current_sense
- R18 pad 2: 2 -> gnd
- R2 pad 2: 2 -> gnd
- R3 pad 1: control-1 -> current_sense
- R3 pad 2: aux2_stage-gate -> gnd
- U1 pad 1: drain -> (no net)
- U1 pad 2: power_in -> (no net)
- U1 pad 3: power_out -> gnd
- U1 pad 4: power_in -> input
- U4 pad 2: 2 -> gnd
- U5 pad 2: 2 -> gnd
- U6 pad 1: pump_stage-drain -> (no net)
- U6 pad 2: power_in -> (no net)
- U6 pad 3: 1-4 -> gnd
- U6 pad 4: power_in -> led_zone1_stage-input
Routing:
- net power_in: track 0.00 -> 491.5 mm, vias 0 -> 2
- net gnd: track 0.00 -> 126.6 mm, vias 0 -> 60
- net v_mcu_5v: track 0.00 -> 94.5 mm
- net control: track 0.00 -> 94.2 mm, vias 0 -> 4
- net control-9: track 0.00 -> 93.5 mm, vias 0 -> 1
- net control-4: track 0.00 -> 77.6 mm, vias 0 -> 1
- net control-10: track 0.00 -> 77.0 mm, vias 0 -> 2
- net control-8: track 0.00 -> 70.2 mm
- net control-5: track 0.00 -> 62.1 mm, vias 0 -> 1
- net control-3: track 0.00 -> 61.2 mm, vias 0 -> 2
- net control-7: track 0.00 -> 52.0 mm, vias 0 -> 2
- net control-6: track 0.00 -> 46.6 mm, vias 0 -> 1
- net 1-3: track 0.00 -> 27.7 mm
- net power_out-7: track 0.00 -> 21.1 mm
- net power_out-4: track 0.00 -> 21.1 mm
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- added copper zone on B.Cu, net gnd
- added copper zone on F.Cu, net gnd
Other:
- board outline added: 150 x 95 mm
